File: statimperium/statimperium.kicad_sch (KiCad schematic)
At the start: 0 parts

Commit message: V1.0.a-1 complete
Parts:
- added Q1: BSS138, Package_TO_SOT_SMD:SOT-23, symbol Transistor_FET:BSS138
- added U3: KLM4G1FETE-B041, eMMC:BGA153_11x10mm_0.15mm, symbol eMMC:KLM4G1FETE-B041
- added U6: SFH617A-1X007T, Package_DIP:SMDIP-4_W9.53mm_Clearance8mm, symbol Isolator:SFH617A-1X007T
Connections:
- new net VCC: U3.E6 (VCC), U3.F5 (VCC), U3.J10 (VCC), U3.K9 (VCC)
- new net VCCQ: U3.C6 (VCCQ), U3.M4 (VCCQ), U3.N4 (VCCQ), U3.P3 (VCCQ), U3.P5 (VCCQ)
- new net VSS: U3.A6 (VSS), U3.C4 (VSS), U3.E7 (VSS), U3.G5 (VSS), U3.H10 (VSS), U3.J5 (VSS), U3.K8 (VSS), U3.N2 (VSS), U3.N5 (VSS), U3.P4 (VSS), U3.P6 (VSS)
Other:
- added sheet MPU (mpu_arch.kicad_sch)
- added sheet Power Management (pwr_management.kicad_sch)
- added sheet memory (memory.kicad_sch)
