File: renodus/renodus.kicad_sch (KiCad schematic)
At the start: 0 parts

Commit message: V1.0.a-1 complete
Parts:
- added AE1: Antenna_Chip, RF_Antenna:AANI-CH-0129-T, symbol Device:Antenna_Chip
- added C1, C12: 2u2, smaller_sizes:0201_universal, symbol Device:C
- added C10, C4, C7, C8: 100n, smaller_sizes:0201_universal, symbol Device:C
- added C11: 0p3, smaller_sizes:0201_universal, symbol Device:C
- added C13, C14, C2: 10u, smaller_sizes:0603_universal, symbol Device:C_Small
- added C15: 2u2, smaller_sizes:0603_universal, symbol Device:C_Small
- added C16, C18: 1u, smaller_sizes:0603_universal, symbol Device:C_Small
- added C17, C19, C20, C21, C23: 100n, smaller_sizes:0201_universal, symbol Device:C_Small
- added C3: 10u, smaller_sizes:0402_universal, symbol Device:C
- added C5: 2n2, smaller_sizes:0201_universal, symbol Device:C
- added C6: 1p5, smaller_sizes:0201_universal, symbol Device:C
- added C9: 2p, smaller_sizes:0201_universal, symbol Device:C
- added D1: LED_ARGB, LED_SMD:LED_Wurth_150044M155260, symbol Device:LED_ARGB
- added FB1: 120R/0.2A, smaller_sizes:0201_universal, symbol Device:FerriteBead_Small
- added H1: MountingHole_Pad, MountingHole:MountingHole_2.2mm_M2_Pad_Via, symbol Mechanical:MountingHole_Pad
- added J1: USB_C_Receptacle_PowerOnly_6P, Connector_USB:USB_C_Receptacle_GCT_USB4125-xx-x-0190_6P_TopMnt_Horizontal, symbol Connector:USB_C_Receptacle_PowerOnly_6P
- added J2: Conn_01x02_Socket, JST_S2B-PH-SM4-TB:JST_S2B-PH-SM4-TB, symbol Connector:Conn_01x02_Socket
- added J3: Conn_ARM_SWD_TagConnect_TC2030, Connector:Tag-Connect_TC2030-IDC-NL_2x03_P1.27mm_Vertical, symbol Connector:Conn_ARM_SWD_TagConnect_TC2030
- added JP1: SHPHLD, Jumper:SolderJumper-2_P1.3mm_Open_RoundedPad1.0x1.5mm, symbol Jumper:SolderJumper_2_Open
- added L1: 4u7, smaller_sizes:0603_universal, symbol Device:L
- added L2: 2n7, smaller_sizes:0201_universal, symbol Device:L
- added L3, L4: 3n5, smaller_sizes:0201_universal, symbol Device:L
- added L5: 2u2, inductor_0806:INDC2016X100N, symbol Device:L_Small
- added R1: 470k, smaller_sizes:0201_universal, symbol Device:R
- added R2, R3, R4: 10k, smaller_sizes:0201_universal, symbol Device:R
- added R5: 50k, smaller_sizes:0201_universal, symbol Device:R
- added SW1: SW_Push, Button_Switch_SMD:SW_SPST_Omron_B3FS-101xP, symbol Switch:SW_Push
- added SW2: SW_Push, Button_Switch_SMD:SW_SPST_CK_KMS2xxGP, symbol Switch:SW_Push
- added TP1: UART_TX, TestPoint:TestPoint_Pad_D1.0mm, symbol Connector:TestPoint
- added TP10: ~{PAIR}, TestPoint:TestPoint_Pad_D0.5mm, symbol Connector:TestPoint
- added TP11: NPMINT, TestPoint:TestPoint_Pad_D0.5mm, symbol Connector:TestPoint
- added TP12: SDA, TestPoint:TestPoint_Pad_D0.5mm, symbol Connector:TestPoint
- added TP13: SCL, TestPoint:TestPoint_Pad_D0.5mm, symbol Connector:TestPoint
- added TP14: SDA_C, TestPoint:TestPoint_Pad_D0.5mm, symbol Connector:TestPoint
- added TP15: SCL_C, TestPoint:TestPoint_Pad_D0.5mm, symbol Connector:TestPoint
- added TP2: UART_RX, TestPoint:TestPoint_Pad_D1.0mm, symbol Connector:TestPoint
- added TP3: CC1, TestPoint:TestPoint_Pad_D0.5mm, symbol Connector:TestPoint
- added TP4: CC2, TestPoint:TestPoint_Pad_D0.5mm, symbol Connector:TestPoint
- added TP5: VBAT, TestPoint:TestPoint_Pad_D0.5mm, symbol Connector:TestPoint
- added TP6: VBUS, TestPoint:TestPoint_Pad_D0.5mm, symbol Connector:TestPoint
- added TP7: VSYS, TestPoint:TestPoint_Pad_D0.5mm, symbol Connector:TestPoint
- added TP8: VBUS_OUT, TestPoint:TestPoint_Pad_D0.5mm, symbol Connector:TestPoint
- added TP9: 3V0, TestPoint:TestPoint_Pad_D0.5mm, symbol Connector:TestPoint
- added U1: nRF54lxx_QDAA, Package_DFN_QFN:QFN-40-1EP_5x5mm_P0.4mm_EP3.6x3.6mm_ThermalVias, symbol MCU_Nordic:nRF54lxx_QDAA
- added U2: NPM1300-QEAA-R, footprints:QFN32_5X5_NOR-L, symbol NPM1300-QEAA-R:NPM1300-QEAA-R
- added U3: SHT4x, Sensor_Humidity:Sensirion_DFN-4_1.5x1.5mm_P0.8mm_SHT4x_NoCentralPad, symbol Sensor_Humidity:SHT4x
- added U4: STCC4, Sensor:STCC4, symbol Sensor_Gas:STCC4
- added Y1: Crystal_GND24_Small, Crystal:Crystal_SMD_2016-4Pin_2.0x1.6mm, symbol Device:Crystal_GND24_Small
- added Y2: Crystal_Small, Crystal:Crystal_SMD_2012-2Pin_2.0x1.2mm, symbol Device:Crystal_Small
- added Z1: 0, smaller_sizes:0201_universal, symbol Device:R
- added Z2: 3n6H, smaller_sizes:0201_universal, symbol Device:R
- added Z3: TBD, smaller_sizes:0201_universal, symbol Device:R
Connections:
- new net: L5.2, U2.5 (SW2)
- new net: C11.1, L4.1, Z1.2, Z2.2
- new net: R1.1, U2.16 (VSET2)
- new net: C9.1, L3.1, L4.2
- new net: C6.1, L2.1, L3.2
- new net: C12.1, C5.1, FB1.2, U1.28 (DECRF), U1.36 (DECA)
- new net: U1.1 (P1.00/XL1), Y2.1
- new net: U1.2 (P1.01/XL2), Y2.2
- new net: L2.2, U1.26 (ANT)
- new net: C1.1, FB1.1, L1.2, U1.38 (DECD)
- new net: L1.1, U1.39 (DCC)
- new net: AE1.1 (FEED), Z1.1, Z3.1
- new net +3V0: C10.1, C17.1, C2.1, C20.1, C21.1, C3.1, C4.1, C7.1, C8.1, J3.1 (VCC), L5.1, R2.1, R3.1, TP9.1, U1.19 (VDD), U1.31 (VDD), U1.40 (VDD), U1.9 (VDD), U2.12 (VDDIO), U2.32 (VOUT2), U3.3 (VDD), U4.6 (VDDIO), U4.7 (VDD)
- new net CC1: J1.A5 (CC1), TP3.1, U2.23 (CC1)
- new net CC2: J1.B5 (CC2), TP4.1, U2.24 (CC2)
- new net GND: C1.2, C10.2, C11.2, C12.2, C13.2, C14.2, C15.2, C16.2, C17.2, C18.2, C19.2, C2.2, C20.2, C21.2, C23.2, C3.2, C4.2, C5.2, C6.2, C7.2, C8.2, C9.2, H1.1, J1.A12 (GND), J1.B12 (GND), J1.S1 (SHIELD), J2.2 (Pin_2), J3.5 (GND), JP1.2 (B), R1.2, R4.2, SW1.1, SW2.1, U1.27 (VSS_PA), U1.37 (VSS), U1.41 (VSS), U2.17 (VSET1), U2.2 (PVSS1), U2.28 (LSIN1/VINLDO1), U2.29 (LSOUT1/VOUTLDO1), U2.30 (LSIN2/VINLDO2), U2.31 (LSOUT2/VOUTLDO2), U2.33 (AVSS), U2.6 (PVSS2), U3.4 (VSS), U4.3 (ADDR), U4.4 (VSS), Y1.2 (G), Y1.4 (G), Z2.1, Z3.2
- new net GPIO0: U2.7 (GPIO0)
- new net GPIO1_PMIC_INT: TP11.1, U1.20 (P0.00), U2.8 (GPIO1)
- new net GPIO2: U2.9 (GPIO2)
- new net GPIO3: U2.10 (GPIO3)
- new net GPIO4: U2.11 (GPIO4)
- new net LED0: D1.2 (RK), U2.27 (LED2)
- new net LED1: D1.3 (GK), U2.26 (LED1)
- new net LED2: D1.4 (BK), U2.25 (LED0)
- new net NTC: R4.1, U2.18 (NTC)
- new net SCL: R2.2, TP13.1, U1.24 (P0.04), U2.14 (SCL), U4.1 (SCL)
- new net SCL_C: TP15.1, U3.2 (SCL), U4.8 (SCL_C)
- new net SDA: R3.2, TP12.1, U1.21 (P0.01), U2.13 (SDA), U4.5 (SDA)
- new net SDA_C: TP14.1, U3.1 (SDA), U4.2 (SDA_C)
- new net SHPHLD: JP1.1 (A), R5.2, U2.15 (SHPHLD)
- new net SWDCLK: J3.4 (SWCLK), U1.23 (SWDCLK)
- new net SWDIO: J3.2 (SWDIO), U1.22 (SWDIO)
- new net UART_RX: TP2.1, U1.17 (P2.07)
- new net UART_TX: TP1.1, U1.18 (P2.08)
- new net VBAT: C15.1, J2.1 (Pin_1), TP5.1, U2.19 (VBAT)
- new net VBUS: C16.1, J1.A9 (VBUS), J1.B9 (VBUS), TP6.1, U2.21 (VBUS)
- new net VBUSOUT: C18.1, TP8.1, U2.22 (VBUSOUT)
- new net VSYS: C13.1, C14.1, D1.1 (A), R5.1, TP7.1, U2.1 (VOUT1), U2.20 (VSYS), U2.4 (PVDD)
- new net XC1: U1.29 (XC1), Y1.1
- new net XC2: U1.30 (XC2), Y1.3
- new net ~{PAIR}: C19.1, SW1.2, TP10.1, U1.3 (P1.02/NFC1)
- new net ~{RESET}: C23.1, J3.3 (~{RESET}), SW2.2, U1.25 (~{RESET})
- no-connect marks 0 -> 19

Commit message: V1.0.a-2
Parts:
- SW2: footprint Button_Switch_SMD:SW_SPST_CK_KMS2xxGP -> Button_Switch_SMD:SW_Push_1P1T_NO_CK_KMR2
- Z2: value 3n6H -> TBD; now not fitted; now left out of the parts list
Changed lines of the file:
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@@
 			)
 		)
-		(property "Footprint" "Button_Switch_SMD:SW_SPST_CK_KMS2xxGP"
+		(property "Footprint" "Button_Switch_SMD:SW_Push_1P1T_NO_CK_KMR2"
 			(at 74.93 46.99 0)
 			(hide yes)
@@
 		(body_style 1)
 		(exclude_from_sim no)
-		(in_bom yes)
-		(on_board yes)
+		(in_bom no)
+		(on_board no)
 		(in_pos_files yes)
-		(dnp no)
+		(dnp yes)
 		(property "Reference" "Z2"
 			(at 41.91 115.57 0)
@@
 			)
 		)
-		(property "Value" "3n6H"
-			(at 40.64 118.11 0)
-			(show_name no)
-			(do_not_autoplace no)
+		(property "Value" "TBD"
+			(at 41.91 118.11 0)
+			(show_name no)
+			(do_not_autoplace no)

Commit message: Small update
Parts:
- AE1: Link (none) -> https://www.digikey.ca/en/products/detail/abracon-llc/AANI-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; Part Num. (none) -> AANI-CH-0129-T
- C1, C12: Link (none) -> https://www.digikey.ca/en/products/detail/murata-electronic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; Part Num. (none) -> GRM033R61A225KE47
- C10, C4, C7, C8: Link (none) -> https://www.digikey.ca/en/products/detail/murata-electronic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; Part Num. (none) -> GRM033Z71A104KE14D
- C11: Link (none) -> https://www.digikey.ca/en/products/detail/murata-electronic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; Part Num. (none) -> GRM0335C1HR30BA01
- C13, C14, C2: Link (none) -> https://www.digikey.ca/en/products/detail/murata-electronic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; Part Num. (none) -> GRM188R61A106ME69J
- C15: Link (none) -> https://www.digikey.ca/en/products/detail/murata-electronic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; Part Num. (none) -> GRM188R61E225KA12D
- C16, C18: Link (none) -> https://www.digikey.ca/en/products/detail/samsung-electro-m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; Part Num. (none) -> CL10A105KP8NNNC
- C17, C19, C20, C21, C23: Link (none) -> https://www.digikey.ca/en/products/detail/tdk/C0603X5R1E104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; Part Num. (none) -> C0603X5R1E104K030BB
- C3: Link (none) -> https://www.digikey.ca/en/products/detail/murata-electronic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; Part Num. (none) -> GRT155C80J106ME13J
- C5: Link (none) -> https://www.digikey.ca/en/products/detail/murata-electronic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; Part Num. (none) -> GRM033R71A222KA01D
- C6: Link (none) -> https://www.digikey.ca/en/products/detail/murata-electronic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; Part Num. (none) -> GJM0335C1E1R5WB01
- C9: Link (none) -> https://www.digikey.ca/en/products/detail/murata-electronic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; Part Num. (none) -> GJM0335C1E2R0WB01
- D1: Link (none) -> https://www.digikey.ca/en/products/detail/w%C3%BCrth-elektr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; Part Num. (none) -> 150044M155260
- FB1: Link (none) -> https://www.digikey.ca/en/products/detail/murata-electronic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; Part Num. (none) -> BLM03AG121SN1D
- H1, JP1: now not fitted
- J1: Link (none) -> https://www.digikey.ca/en/products/detail/gct/USB4125-GF-A/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; Part Num. (none) -> USB4125-GF-A
- J2: Link (none) -> https://www.digikey.ca/en/products/detail/jst-sales-america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; Part Num. (none) -> S2B-PH-SM4-TB
- L1: Link (none) -> https://www.digikey.ca/en/products/detail/tdk/MLZ1608M4R7WT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; Part Num. (none) -> MLZ1608M4R7WT000
- L2: Link (none) -> https://www.digikey.ca/en/products/detail/murata-electronic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; Part Num. (none) -> LQP03HQ2N7B02
- L3, L4: Link (none) -> https://www.digikey.ca/en/products/detail/murata-electronic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; Part Num. (none) -> LQP03HQ3N5B02
- L5: Link (none) -> https://www.digikey.ca/en/products/detail/samsung-electro-m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; Part Num. (none) -> CIGT201610EH2R2MNE
- R1: Link (none) -> https://www.digikey.ca/en/products/detail/panasonic-industr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; Part Num. (none) -> ERJ-1GNF4703C
- R2, R3, R4: Link (none) -> https://www.digikey.ca/en/products/detail/yageo/RC0201FR-07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; Part Num. (none) -> RC0201FR-0710KL
- R5: value 50k -> 51k; Link (none) -> https://www.digikey.ca/en/products/detail/yageo/RC0201JR-07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; Part Num. (none) -> RC0201JR-0751KL
- SW1: Link (none) -> https://www.digikey.ca/en/products/detail/aratas-america-ll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; Part Num. (none) -> B3FS-1012P
- SW2: Link (none) -> https://www.digikey.ca/en/products/detail/c-k/KMR231G-LFS/5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; Part Num. (none) -> KMR231G LFS
- TP1, TP10, TP11, TP12, TP13, TP14, TP15, TP2, TP3, TP4, TP5, TP6, TP7, TP8, TP9: now left out of the parts list
- U1: Link (none) -> https://www.digikey.ca/en/products/detail/nordic-semiconduc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; Part Num. (none) -> NRF54L10-QDAA-R7
- U2: DigiKey_Part_Number 4823-NPM1300-QEAA-RCT-ND -> (none); Link (none) -> https://www.digikey.ca/en/products/detail/nordic-semiconduc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; Part Num. (none) -> NPM1300-QEAA-R7
- U3: Link (none) -> https://www.digikey.ca/en/products/detail/sensirion-ag/SHT4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; Part Num. (none) -> SHT41A-AW1B-R3
- U4: Link (none) -> https://www.digikey.ca/en/products/detail/sensirion-ag/STCC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; Part Num. (none) -> STCC4-D-R3
- Y1: Link (none) -> https://www.digikey.ca/en/products/detail/kyocera-avx/CX201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; Part Num. (none) -> CX2016DB32000D0WZRC1
- Y2: value Crystal_Small -> 32.768kHz; Link (none) -> https://www.digikey.ca/en/products/detail/kyocera-avx/CX201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; Part Num. (none) -> 9HT11-32.768KDZC-T
- Z1: Link (none) -> https://www.digikey.ca/en/products/detail/yageo/RC0201JR-07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; Part Num. (none) -> RC0201JR-070RL
