File: renodus/renodus.kicad_pcb (KiCad board)
At the start: 4 copper layers, 40 x 40 mm, 66 parts, among them J1 USB_C_Receptacle_PowerOnly_6P, J2 Conn_01x02_Socket, J3 Conn_ARM_SWD_TagConnect_TC2030, SW1 SW_Push, SW2 SW_Push, U1 nRF54lxx_QDAA, U2 NPM1300-QEAA-R, U3 SHT4x, U4 STCC4, Y1 Crystal_GND24_Small, Y2 Crystal_Small

Commit message: Button Position Modified
Parts:
- moved C19 3.54 mm to (175.8, 84.6)
- moved D1 3.54 mm to (175.8, 90.9)
- moved SW1 3.54 mm to (172.6, 87.7)
- moved TP10 3.54 mm to (178.8, 88.2)
Routing:
- net /~{PAIR}: track 25.2 -> 21.1 mm
- net /LED2: track 37.1 -> 35.2 mm
- net VSYS: track 33.8 -> 31.9 mm
- net /LED0: track 35.9 -> 34.1 mm
- net /LED1: track 36.0 -> 34.2 mm
- net GND: track 55.0 -> 55.6 mm, vias 254 -> 255
Changed lines of the file:
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@@
 	(footprint "Button_Switch_SMD:SW_SPST_Omron_B3FS-101xP"
 		(layer "F.Cu")
-		(at 170.109279 85.196965 45)
+		(at 172.609279 87.696965 45)
 		(descr "Surface Mount Tactile Switch for High-Density Mounting, 4.3mm height, https://omronfs.omron.com/en_US/ecb/products/pdf/en-b3fs.pdf")
 		(tags "Tactile Switch")
@@
 	(footprint "TestPoint:TestPoint_Pad_D0.5mm"
 		(layer "F.Cu")
-		(at 176.28699 85.741405 180)
+		(at 178.78699 88.241405 180)
 		(descr "SMD pad as test Point, diameter 1.0mm")
 		(tags "test point SMD pad")
@@
 	(footprint "LED_SMD:LED_Wurth_150044M155260"
 		(layer "F.Cu")
-		(at 173.29126 88.378946 45)
+		(at 175.79126 90.878946 45)
 		(descr "Wurth Common anode RGB LED, SMD, 0404, 1x1x1.65mm, https://www.we-online.com/catalog/datasheet/150044M155260.pdf")
 		(tags "LED RGB ARGB ")
@@
 	(footprint "smaller_sizes:0201_universal"
 		(layer "F.Cu")
-		(at 173.289424 82.143839 135)
+		(at 175.789424 84.643839 135)
 		(tags "GRM0335C1H100FA01D ")
 		(property "Reference" "C19"
@@
 			(polygon
 				(pts
-					(xy 173.253503 82.251602) (xy 173.181661 82.17976) (xy 173.325345 82.036076) (xy 173.397187 82.107918)
+					(xy 175.753503 84.751602) (xy 175.681661 84.67976) (xy 175.825345 84.536076) (xy 175.897187 84.607918)
 				)
 			)
@@
 	)
 	(gr_text "HOLD TO PAIR"
-		(at 174.08699 81.191405 315)
+		(at 176.58699 83.691405 315)
 		(layer "F.SilkS")
 		(effects
@@
 	)
 	(segment
+		(start 174.528696 83.983111)
+		(end 174.528696 83.959528)
+		(width 0.15)
+		(layer "F.Cu")
+		(net "GND")
+	)
+	(segment
 		(start 184.33699 108.316304)
 		(end 184.33699 107.691403)
@@
 	)
 	(segment
+		(start 174.528696 83.959528)
+		(end 174.528696 83.383111)
+		(width 0.15)
+		(layer "F.Cu")
+		(net "GND")
+	)
+	(segment
 		(start 187.633305 87.801138)
 		(end 186.888721 87.056554)
@@
 	)
 	(via
-		(at 166.43699 82.35688)
+		(at 166.48699 82.191405)
+		(size 0.5)
+		(drill 0.25)
+		(layers "F.Cu" "B.Cu")
+		(free yes)
+		(net "GND")
+	)
+	(via
+		(at 167.68699 86.391405)
 		(size 0.5)
 		(drill 0.25)
@@
 	)
 	(via
-		(at 166.43699 85.991405)
+		(at 166.48699 85.791405)
 		(size 0.5)
 		(drill 0.25)
@@
 	)
 	(via
-		(at 166.43699 85.35688)
+		(at 166.48699 85.191405)
 		(size 0.5)
 		(drill 0.25)
@@
 	)
 	(via
-		(at 166.43699 81.741405)
+		(at 166.48699 81.591405)
 		(size 0.5)
 		(drill 0.25)
@@
 	)
 	(via
-		(at 172.63699 81.491405)
+		(at 175.13699 83.991405)
 		(size 0.5)
 		(drill 0.25)
@@
 	)
 	(via
-		(at 166.43699 82.95688)
+		(at 166.48699 82.791405)
 		(size 0.5)
 		(drill 0.25)
@@
 	)
 	(via
-		(at 167.03699 81.70688)
+		(at 167.08699 81.591405)
 		(size 0.5)
 		(drill 0.25)
@@
 	)
 	(via
-		(at 166.43699 84.15688)
+		(at 166.48699 83.991405)
 		(size 0.5)
 		(drill 0.25)
@@
 	)
 	(via
-		(at 166.43699 83.55688)
+		(at 166.48699 83.391405)
 		(size 0.5)
 		(drill 0.25)
@@
 	)
 	(via
-		(at 167.63699 86.30688)
+		(at 167.08699 86.391405)
 		(size 0.5)
 		(drill 0.25)
@@
 	)
 	(via
-		(at 167.63699 81.70688)
+		(at 167.68699 81.591405)
 		(size 0.5)
 		(drill 0.25)
@@
 	)
 	(via
-		(at 167.03699 86.30688)
+		(at 166.48699 86.391405)
 		(size 0.5)
 		(drill 0.25)
@@
 	)
 	(via
-		(at 166.43699 84.75688)
+		(at 166.48699 84.591405)
 		(size 0.5)
 		(drill 0.25)
@@
 	)
 	(segment
-		(start 172.725575 89.47999)
-		(end 172.725575 88.378946)
-		(width 0.2)
-		(layer "F.Cu")
-		(net "VSYS")
-	)
-	(segment
 		(start 179.98699 98.941405)
 		(end 179.98699 99.282603)
@@
 	)
 	(segment
-		(start 173.18699 89.941405)
-		(end 172.725575 89.47999)
+		(start 178.533436 104.387851)
+		(end 178.53699 104.391405)
 		(width 0.2)
 		(layer "F.Cu")
@@
 	)
 	(segment
-		(start 178.533436 104.387851)
-		(end 178.53699 104.391405)
+		(start 175.225575 91.97999)
+		(end 175.225575 90.878946)
 		(width 0.2)
 		(layer "F.Cu")
@@
 	)
 	(via
-		(at 173.18699 89.941405)
+		(at 175.225575 91.97999)
 		(size 0.5)
 		(drill 0.25)
@@
 	)
 	(segment
-		(start 173.18699 89.941405)
-		(end 173.18699 101.641405)
+		(start 173.18699 101.641405)
+		(end 175.93699 104.391405)
 		(width 0.2)
 		(layer "In2.Cu")
@@
 	)
 	(segment
-		(start 178.58699 104.341405)
+		(start 175.93699 104.391405)
 		(end 178.53699 104.391405)
-		(width 0.15)
+		(width 0.2)
 		(layer "In2.Cu")
 		(net "VSYS")
 	)
 	(segment
-		(start 175.93699 104.391405)
+		(start 178.58699 104.341405)
 		(end 178.53699 104.391405)
-		(width 0.2)
+		(width 0.15)
 		(layer "In2.Cu")
 		(net "VSYS")
@@
 	)
 	(segment
-		(start 173.18699 101.641405)
-		(end 175.93699 104.391405)
+		(start 175.225575 91.97999)
+		(end 175.225575 92.00282)
+		(width 0.2)
+		(layer "In2.Cu")
+		(net "VSYS")
+	)
+	(segment
+		(start 173.18699 94.041405)
+		(end 173.18699 101.641405)
 		(width 0.2)
 		(layer "In2.Cu")
@@
 	)
 	(segment
+		(start 175.225575 92.00282)
+		(end 173.18699 94.041405)
+		(width 0.2)
+		(layer "In2.Cu")
+		(net "VSYS")
+	)
+	(segment
 		(start 178.53699 104.391405)
 		(end 178.53699 104.741405)
@@
 	)
 	(segment
-		(start 173.78699 101.341405)
-		(end 173.78699 89.440361)
+		(start 182.58699 109.941405)
+		(end 181.336991 108.691406)
 		(width 0.2)
 		(layer "F.Cu")
@@
 	)
 	(segment
-		(start 182.58699 109.941405)
-		(end 181.336991 108.691406)
+		(start 185.68699 109.941405)
+		(end 182.58699 109.941405)
 		(width 0.2)
 		(layer "F.Cu")
@@
 	)
 	(segment
-		(start 185.68699 109.941405)
-		(end 182.58699 109.941405)
+		(start 175.78699 91.448901)
+		(end 175.79126 91.444631)
 		(width 0.2)
 		(layer "F.Cu")
@@
 	)
 	(segment
-		(start 173.29126 88.945675)
-		(end 173.29126 88.944631)
+		(start 173.78699 101.341405)
+		(end 173.78699 94.541407)
 		(width 0.2)
 		(layer "F.Cu")
@@
 	)
 	(segment
-		(start 173.78699 89.440361)
-		(end 173.29126 88.944631)
+		(start 173.78699 94.541407)
+		(end 175.78699 92.541407)
+		(width 0.2)
+		(layer "F.Cu")
+		(net "/LED2")
+	)
+	(segment
+		(start 175.78699 92.541407)
+		(end 175.78699 91.448901)
 		(width 0.2)
 		(layer "F.Cu")
@@
 	)
 	(segment
-		(start 185.98699 109.541405)
-		(end 182.68699 109.541405)
+		(start 174.28699 94.741409)
+		(end 176.38699 92.641409)
+		(width 0.2)
+		(layer "F.Cu")
+		(net "/LED1")
+	)
+	(segment
+		(start 176.38699 92.641409)
+		(end 176.38699 90.908991)
 		(width 0.2)
 		(layer "F.Cu")
@@
 	)
 	(segment
-		(start 174.28699 88.808991)
-		(end 173.856945 88.378946)
+		(start 174.28699 101.741405)
+		(end 174.28699 94.741409)
+		(width 0.2)
+		(layer "F.Cu")
+		(net "/LED1")
+	)
+	(segment
+		(start 185.98699 109.541405)
+		(end 182.68699 109.541405)
 		(width 0.2)
 		(layer "F.Cu")
@@
 	)
 	(segment
-		(start 174.28699 101.741405)
-		(end 174.28699 88.808991)
+		(start 176.38699 90.908991)
+		(end 176.356945 90.878946)
 		(width 0.2)
 		(layer "F.Cu")
@@
 	)
 	(segment
-		(start 174.78699 88.341405)
-		(end 174.258846 87.813261)
+		(start 186.28699 109.141405)
+		(end 182.78699 109.141405)
 		(width 0.2)
 		(layer "F.Cu")
@@
 	)
 	(segment
-		(start 174.258846 87.813261)
-		(end 173.29126 87.813261)
+		(start 182.336989 108.691404)
+		(end 182.336989 108.316305)
 		(width 0.2)
 		(layer "F.Cu")
@@
 	)
 	(segment
-		(start 186.28699 109.141405)
-		(end 182.78699 109.141405)
+		(start 176.98699 90.741405)
+		(end 176.558846 90.313261)
 		(width 0.2)
 		(layer "F.Cu")
@@
 	)
 	(segment
-		(start 182.336989 108.691404)
-		(end 182.336989 108.316305)
+		(start 174.78699 102.141405)
+		(end 174.78699 94.941407)
+		(width 0.2)
+		(layer "F.Cu")
+		(net "/LED0")
+	)
+	(segment
+		(start 176.98699 92.741407)
+		(end 176.98699 90.741405)
 		(width 0.2)
 		(layer "F.Cu")
@@
 	)
 	(segment
-		(start 174.78699 102.141405)
-		(end 174.78699 88.341405)
+		(start 176.558846 90.313261)
+		(end 175.79126 90.313261)
+		(width 0.2)
+		(layer "F.Cu")
+		(net "/LED0")
+	)
+	(segment
+		(start 174.78699 94.941407)
+		(end 176.98699 92.741407)
 		(width 0.2)
 		(layer "F.Cu")
@@
 	)
 	(segment
-		(start 178.73699 88.191405)
-		(end 174.528696 83.983111)
+		(start 178.78699 88.241405)
+		(end 177.028696 86.483111)
 		(width 0.15)
 		(layer "F.Cu")
@@
 	)
 	(segment
-		(start 174.528696 83.983111)
-		(end 174.528696 83.959528)
-		(width 0.15)
-		(layer "F.Cu")
-		(net "/~{PAIR}")
-	)
-	(segment
 		(start 178.73699 96.891405)
 		(end 178.73699 88.191405)
@@
 	)
 	(segment
-		(start 174.528696 83.383111)
-		(end 173.48699 82.341405)
+		(start 177.028696 85.883111)
+		(end 175.98699 84.841405)
 		(width 0.15)
 		(layer "F.Cu")
@@
 		(width 0.15)
 		(layer "F.Cu")
-		(net "/~{PAIR}")
-	)
-	(segment
-		(start 174.528696 83.959528)
-		(end 174.528696 83.383111)
-		(width 0.15)
-		(layer "F.Cu")

Commit message: V1.0.a-2
Parts:
- added G***: LOGO, renodus_icon:renodus_icon, B.Cu at (195.0, 86.5)
- C23: moved to B.Cu
- SW2: footprint Button_Switch_SMD:SW_SPST_CK_KMS2xxGP -> Button_Switch_SMD:SW_Push_1P1T_NO_CK_KMR2; moved to B.Cu
- moved SW2 18.2 mm to (176.9, 84.6), turned to 90 degrees
- moved C23 13.6 mm to (176.4, 87.8)
- moved J1 0.10 mm to (183.1, 114.8)
Routing:
- net /~{PAIR}: track 21.1 -> 29.1 mm
- net /~{RESET}: track 47.3 -> 46.6 mm, vias 3 -> 2
- net GND: vias 255 -> 256

Commit message: Small update
Changed lines of the file:
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@@
 			(effects
 				(font
-					(size 1 1)
-					(thickness 0.15)
+					(size 0.5 0.5)
+					(thickness 0.125)
 				)
 			)
@@
 	)
 	(zone
-		(net "+3V0")
-		(layer "F.Cu")
-		(hatch none 0.1)
-		(priority 30000)
-		(attr
-			(teardrop
-				(type padvia)
-			)
-		)
-		(connect_pads yes
-			(clearance 0)
-		)
-		(min_thickness 0.0254)
-		(fill yes
-			(island_removal_mode 1)
-		)
-		(polygon
-			(pts
-				(xy 189.591794 106.341405) (xy 189.591794 106.741405) (xy 190.038217 106.786601) (xy 190.092794 106.541405)
-				(xy 190.038217 106.296209)
-			)
-		)
-	)
-	(zone
 		(layer "F.Cu")
 		(name "VBAT_BTM")
@@
 			)
 		)
+	)
+	(zone
+		(net "+3V0")
+		(layer "F.Cu")
+		(hatch none 0.1)
+		(priority 30000)
+		(attr
+			(teardrop
+				(type padvia)
+			)
+		)
+		(connect_pads yes
+			(clearance 0)
+		)
+		(min_thickness 0.0254)
+		(fill yes
+			(island_removal_mode 1)
+		)
+		(polygon
+			(pts
+				(xy 189.591794 106.341405) (xy 189.591794 106.741405) (xy 190.038217 106.786601) (xy 190.092794 106.541405)
+				(xy 190.038217 106.296209)
+			)
+		)

Commit message: Fixed Gerbers
Parts:
- removed Z2: 3n6H, smaller_sizes:0201_universal
- R5: value 50k -> 51k
- Y2: value Crystal_Small -> 32.768kHz
